Commit message: Change the elevator(where sensors) and gps location (in urdf)

File: rbcar_description/robots/versions/rbcar_roborder.urdf.xacro (robot description, xacro)
@@ -61,8 +61,8 @@
 	</xacro:sensor_imu_hector>
 	<xacro:sensor_gps prefix="$(arg prefix)gps" parent="$(arg prefix)base_link" gps_latitude="$(arg gps_latitude)" gps_longitude="$(arg gps_longitude)" update_rate="20" >
-		<origin xyz="0.0 0 1.5" rpy="0 0 0"/>
+		<origin xyz="0.0 0 0.0" rpy="0 0 0"/>
 	</xacro:sensor_gps>
   <xacro:elevator parent="$(arg prefix)base_link" prefix="$(arg prefix)">
-		<origin xyz="0.0 0.0 0.6" rpy="0 0 0"/>
+		<origin xyz="0.8 0.0 0.6" rpy="0 0 0"/>
 	</xacro:elevator>
   <xacro:sensor_axis_q8641 prefix="$(arg prefix)front_ptz_camera" parent="$(arg prefix)elevator_link" far="300" near="0.08">

Commit message: Change the gps coordinates

File: rbcar_description/robots/versions/rbcar_roborder.urdf.xacro (robot description, xacro)
@@ -61,5 +61,5 @@
 	</xacro:sensor_imu_hector>
 	<xacro:sensor_gps prefix="$(arg prefix)gps" parent="$(arg prefix)base_link" gps_latitude="$(arg gps_latitude)" gps_longitude="$(arg gps_longitude)" update_rate="20" >
-		<origin xyz="0.0 0 0.0" rpy="0 0 0"/>
+		<origin xyz="0.0 0 1.5" rpy="0 0 0"/>
 	</xacro:sensor_gps>
   <xacro:elevator parent="$(arg prefix)base_link" prefix="$(arg prefix)">

Commit message: Add lidar and proximity sensor (range)

File: rbcar_description/robots/versions/rbcar_roborder.urdf.xacro (robot description, xacro)
@@ -9,5 +9,5 @@
 	<xacro:include filename="$(find rbcar_description)/urdf/bases/rbcar_base.urdf.xacro" />
 	<!-- Import Robotnik CAR wheels -->
-	<!--xacro:include filename="$(find rbcar_description)/urdf/wheels/suspension_wheel_v3.urdf.xacro" /-->
+	<!-- xacro:include filename="$(find rbcar_description)/urdf/wheels/suspension_wheel_v3.urdf.xacro" / -->
   <xacro:include filename="$(find rbcar_description)/urdf/wheels/suspension_wheel_v2.urdf.xacro" />
 	<xacro:include filename="$(find rbcar_description)/urdf/structures/elevator.urdf.xacro" />
@@ -51,7 +51,7 @@
                     lr_reflect="-1" fr_reflect="-1" parent="$(arg prefix)base_link" />
 	<!-- SENSORS -->
-  <!--xacro:sensor_benewake_ce30d prefix="$(arg prefix)front_3d_lidar" parent="$(arg prefix)base_link" gpu="$(arg gpu)">
+  <!-- <xacro:sensor_benewake_ce30d prefix="$(arg prefix)front_3d_lidar" parent="$(arg prefix)base_link" gpu="$(arg gpu)">
       <origin xyz="2.155 0.0 0.236" rpy="0 0 0"/>
-  </xacro:sensor_benewake_ce30d-->
+  </xacro:sensor_benewake_ce30d> -->
   <!--xacro:sensor_rubedos_viper prefix="$(arg prefix)viper" parent="$(arg prefix)base_link">
       <origin xyz="1.289 0.0 1.354" rpy="0 0.0 0.0"/>
@@ -69,7 +69,10 @@
     <origin xyz="0 0 0" rpy="0 0 0"/>
   </xacro:sensor_axis_q8641>
-  <!--xacro:sensor_rslidar_16 prefix="$(arg prefix)top_3d_laser" parent="$(arg prefix)base_link"  gpu="$(arg gpu)">
+  <xacro:sensor_rslidar_16 prefix="$(arg prefix)top_3d_laser" parent="$(arg prefix)base_link"  gpu="$(arg gpu)">
     <origin xyz="1.163 0.0 1.602" rpy="0 0.2637 0"/>
-  </xacro:sensor_rslidar_16-->
+  </xacro:sensor_rslidar_16>
+  <xacro:sensor_teraranger_duo prefix="$(arg prefix)sonar" parent="$(arg prefix)base_link" min_angle="-0.02618" max_angle="0.02618">
+    <origin xyz="2.5 0 0" rpy="0 0 0"/>
+  </xacro:sensor_teraranger_duo>
 <gazebo>
 <plugin name="ground_truth_controller" filename="librobotnik_gazebo_ground_truth_odom.so">

Commit message: Change the sonar position

File: rbcar_description/robots/versions/rbcar_roborder.urdf.xacro (robot description, xacro)
@@ -73,5 +73,5 @@
   </xacro:sensor_rslidar_16>
   <xacro:sensor_teraranger_duo prefix="$(arg prefix)sonar" parent="$(arg prefix)base_link" min_angle="-0.02618" max_angle="0.02618">
-    <origin xyz="2.5 0 0" rpy="0 0 0"/>
+    <origin xyz="2.3 0 0.2" rpy="0 0 0"/>
   </xacro:sensor_teraranger_duo>
 <gazebo>
