Commit message: Update wheel urdf for the same rotational direction of right and left wheels

File: rbcar_description/urdf/wheels/suspension_wheel_v2.urdf.xacro (robot description, xacro)
@@ -7,6 +7,6 @@
        axle_length. -->
   <xacro:property name="hub_dia" value="0.235"/>
-  <xacro:property name="tire_dia" value="0.634"/>
-  <xacro:property name="tire_width" value="0.322"/>
+  <xacro:property name="tire_dia" value="0.639"/>
+  <xacro:property name="tire_width" value="0.245"/>
   <xacro:property name="hex_hub_depth" value="0.120"/> <!-- or +0.072 -->
   <xacro:property name="wheel_mass" value="8.0"/>   <!-- check -->
@@ -15,7 +15,7 @@
        from a U joint to the corresponding hex hub. wheel_travel is the
        vertical wheel travel. -->
-  <xacro:property name="wheelbase" value="1.83"/>
+  <xacro:property name="wheelbase" value="1.83323"/>
   <!--xacro:property name="hex_hub_dist" value="1.2385"/-->  <!-- 1.127 0.742 0.900 check -->
-  <xacro:property name="axle_length" value="0.120"/>
+  <xacro:property name="axle_length" value="0.12"/>
   <xacro:property name="wheel_travel" value="0.1"/>
   <xacro:property name="shock_z_offset" value="0.05"/>
@@ -30,6 +30,6 @@
   <xacro:property name="wheel_joint_damping" value="0.2" />
   <xacro:property name="wheel_joint_friction" value="0.7" />
-  <xacro:property name="suspension_joint_damping" value="0.2" />
-  <xacro:property name="suspension_joint_friction" value="0.7" />
+  <xacro:property name="suspension_joint_damping" value="0.1" />
+  <xacro:property name="suspension_joint_friction" value="0.1" />
   <!-- axle eff limit = 2 * stall_torque
        as a function of the max gradient (15%) with overall max payload (600Kg) * wheel_radius
@@ -77,10 +77,10 @@
       <child link="${child}"/>
       <xacro:if value="${fr_prefix=='front'}">
-        <xacro:property name="hex_hub_dist" value="1.03802"/>
+        <xacro:property name="hex_hub_dist" value="1.45802"/>
       </xacro:if>
       <xacro:if value="${fr_prefix=='rear'}">
-        <xacro:property name="hex_hub_dist" value="1.2385"/>
-      </xacro:if>
-      <origin xyz="${fr_reflect * wheelbase / 2 + 0.917}
+        <xacro:property name="hex_hub_dist" value="1.45802"/>
+      </xacro:if>
+      <origin xyz="${fr_reflect * wheelbase / 2 + 1}
                    ${lr_reflect * ((hex_hub_dist / 2) - axle_length)}
                    ${(wheel_travel / 2) - shock_z_offset}"/>
@@ -123,5 +123,10 @@
       <child link="${lr_prefix}_${fr_prefix}_wheel"/>
       <origin rpy="-${degrees_90} 0 0"/>
+      <xacro:if value="${lr_reflect == 1}">
+      <axis xyz="0 0 -1"/>
+      </xacro:if>
+      <xacro:if value="${lr_reflect == -1}">
       <axis xyz="0 0 1"/>
+      </xacro:if>
       <limit effort="${axle_eff_limit}" velocity="${axle_vel_limit}"/>
       <joint_properties damping="${wheel_joint_damping}" friction="${wheel_joint_friction}"/>
@@ -192,13 +197,14 @@
       <parent link="${lr_prefix}_steering_link"/>
       <child link="${lr_prefix}_${fr_prefix}_axle_carrier"/>
-      <axis xyz="0 0 1"/>
       <xacro:if value="${lr_reflect == 1}"> <!-- this applies if we are setting the left wheel -->
+        <axis xyz="0 0 1"/>
         <limit lower="${-degrees_34}" upper="${degrees_45}"
              effort="${servo_stall_torque}" velocity="${servo_no_load_speed}"/>
         </xacro:if>
-      <xacro:unless value="${lr_reflect == 1}"> <!-- this applies if we are setting the right wheel -->
+      <xacro:if value="${lr_reflect == -1}"> <!-- this applies if we are setting the right wheel -->
+        <axis xyz="0 0 -1"/>
         <limit lower="${-degrees_45}" upper="${degrees_34}"
              effort="${servo_stall_torque}" velocity="${servo_no_load_speed}"/>
-      </xacro:unless>
+      </xacro:if>
     </joint>
     <transmission name="${lr_prefix}_steering_trans">

Commit message: Hot fix

File: rbcar_description/urdf/wheels/suspension_wheel_v2.urdf.xacro (robot description, xacro)
@@ -124,8 +124,8 @@
       <origin rpy="-${degrees_90} 0 0"/>
       <xacro:if value="${lr_reflect == 1}">
+      <axis xyz="0 0 1"/>
+      </xacro:if>
+      <xacro:if value="${lr_reflect == -1}">
       <axis xyz="0 0 -1"/>
-      </xacro:if>
-      <xacro:if value="${lr_reflect == -1}">
-      <axis xyz="0 0 1"/>
       </xacro:if>
       <limit effort="${axle_eff_limit}" velocity="${axle_vel_limit}"/>
@@ -197,11 +197,12 @@
       <parent link="${lr_prefix}_steering_link"/>
       <child link="${lr_prefix}_${fr_prefix}_axle_carrier"/>
+        <axis xyz="0 0 -1"/>
       <xacro:if value="${lr_reflect == 1}"> <!-- this applies if we are setting the left wheel -->
-        <axis xyz="0 0 1"/>
+        <!-- <axis xyz="0 0 1"/> -->
         <limit lower="${-degrees_34}" upper="${degrees_45}"
              effort="${servo_stall_torque}" velocity="${servo_no_load_speed}"/>
         </xacro:if>
       <xacro:if value="${lr_reflect == -1}"> <!-- this applies if we are setting the right wheel -->
-        <axis xyz="0 0 -1"/>
+        <!-- <axis xyz="0 0 1"/> -->
         <limit lower="${-degrees_45}" upper="${degrees_34}"
              effort="${servo_stall_torque}" velocity="${servo_no_load_speed}"/>

Commit message: change the turning

File: rbcar_description/urdf/wheels/suspension_wheel_v2.urdf.xacro (robot description, xacro)
@@ -197,5 +197,5 @@
       <parent link="${lr_prefix}_steering_link"/>
       <child link="${lr_prefix}_${fr_prefix}_axle_carrier"/>
-        <axis xyz="0 0 -1"/>
+        <axis xyz="0 0 1"/>
       <xacro:if value="${lr_reflect == 1}"> <!-- this applies if we are setting the left wheel -->
         <!-- <axis xyz="0 0 1"/> -->
